File: Kicad/ESP32-aqs/ESP32-aqs.kicad_pcb (KiCad board)
At the start: 2 copper layers, 20 parts, among them J1 UART Connector, J2 Conn SEN55, U1 LD1117S33TR_SOT223, U2 ESP32-WROOM-32, U4 SX1276S8S+T-X1

Commit message: Add files via upload
Parts:
- added J3: ufl connector, Connector_Coaxial:U.FL_Molex_MCRF_73412-0110_Vertical, F.Cu at (180.3, 105.4)
- added U3: SGP41-D-R4, Library:SGP41, F.Cu at (186.1, 104.4)
Connections:
- U4 pad 9: unconnected-(U4-Pad9) -> Net-(J3-Pad1)
Changed lines of the file:
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@@
   (net 38 "MOSI")
   (net 39 "unconnected-(U4-Pad7)")
-  (net 40 "unconnected-(U4-Pad9)")
+  (net 40 "Net-(J3-Pad1)")
   (net 41 "unconnected-(U4-Pad11)")
   (net 42 "unconnected-(U4-Pad12)")
@@
       (rotate (xyz 0 0 0))
     )
+  )
+  (footprint "Library:SGP41" (layer "F.Cu")
+    (at 186.115 104.38)
+    (property "MANUFACTURER" "Sensirion")
+    (property "MAXIMUM_PACKAGE_HEIGHT" "0.95 mm")
+    (property "PARTREV" "1.0")
+    (property "STANDARD" "Manufacturer Recommendations")
+    (property "Sheetfile" "ESP32-aqs.kicad_sch")
+    (property "Sheetname" "")
+    (attr smd)
+    (fp_text reference "U3" (at 0.357 -2.0764) (layer "F.SilkS")
+      (effects (font (size 0.64 0.64) (thickness 0.15)))
+    )
+    (fp_text value "SGP41-D-R4" (at 4.421 2.0764) (layer "F.Fab")
+      (effects (font (size 0.64 0.64) (thickness 0.15)))
+    )
+    (fp_poly (pts
+        (xy -0.225 -0.75)
+        (xy 0.525 -0.75)
+        (xy 0.525 0.75)
+        (xy -0.525 0.75)
+        (xy -0.525 -0.45)
+      ) (layer "F.Paste") (width 0.01) (fill solid))
+    (fp_line (start -1.22 -1.32) (end 1.22 -1.32) (layer "F.SilkS") (width 0.127))
+    (fp_line (start 1.22 1.32) (end -1.22 1.32) (layer "F.SilkS") (width 0.127))
+    (fp_circle (center -2.05 -0.8) (end -1.95 -0.8) (layer "F.SilkS") (width 0.2) (fill none))
+    (fp_poly (pts
+        (xy -0.675 0.9)
+        (xy -0.675 -0.58)
+        (xy -0.355 -0.9)
+        (xy 0.675 -0.9)
+        (xy 0.675 0.9)
+      ) (layer "F.Mask") (width 0.01) (fill solid))
+    (fp_line (start -1.675 1.47) (end 1.675 1.47) (layer "F.CrtYd") (width 0.05))
+    (fp_line (start 1.675 1.47) (end 1.675 -1.47) (layer "F.CrtYd") (width 0.05))
+    (fp_line (start 1.675 -1.47) (end -1.675 -1.47) (layer "F.CrtYd") (width 0.05))
+    (fp_line (start -1.675 -1.47) (end -1.675 1.47) (layer "F.CrtYd") (width 0.05))
+    (fp_line (start 1.22 1.22) (end -1.22 1.22) (layer "F.Fab") (width 0.127))
+    (fp_line (start -1.22 1.22) (end -1.22 -1.22) (layer "F.Fab") (width 0.127))
+    (fp_line (start -1.22 -1.22) (end 1.22 -1.22) (layer "F.Fab") (width 0.127))
+    (fp_line (start 1.22 -1.22) (end 1.22 1.22) (layer "F.Fab") (width 0.127))
+    (fp_circle (center -2.05 -0.8) (end -1.95 -0.8) (layer "F.Fab") (width 0.2) (fill none))
+    (pad "1" smd rect (at -1.15 -0.8) (size 0.55 0.4) (layers "F.Cu" "F.Paste" "F.Mask")
+      (net 3 "+3V3") (pinfunction "VDD") (pintype "power_in"))
+    (pad "2" smd rect (at -1.15 0) (size 0.55 0.4) (layers "F.Cu" "F.Paste" "F.Mask")
+      (net 2 "GND") (pinfunction "VSS") (pintype "power_in"))
+    (pad "3" smd rect (at -1.15 0.8) (size 0.55 0.4) (layers "F.Cu" "F.Paste" "F.Mask")
+      (net 8 "SDA") (pinfunction "SDA") (pintype "bidirectional"))
+    (pad "4" smd rect (at 1.15 0.8) (size 0.55 0.4) (layers "F.Cu" "F.Paste" "F.Mask")
+      (net 2 "GND") (pinfunction "N/A") (pintype "passive"))
+    (pad "5" smd rect (at 1.15 0) (size 0.55 0.4) (layers "F.Cu" "F.Paste" "F.Mask")
+      (net 3 "+3V3") (pinfunction "VDDH") (pintype "power_in"))
+    (pad "6" smd rect (at 1.15 -0.8) (size 0.55 0.4) (layers "F.Cu" "F.Paste" "F.Mask")
+      (net 9 "SCL") (pinfunction "SCL") (pintype "bidirectional"))
+    (pad "7" smd custom (at 0 0) (size 0.5 0.5) (layers "F.Cu")
+      (net 2 "GND") (pinfunction "EXP") (pintype "power_in") (zone_connect 0)
+      (options (clearance outline) (anchor rect))
+      (primitives
+        (gr_poly (pts
+            (xy -0.325 -0.85)
+            (xy 0.625 -0.85)
+            (xy 0.625 0.85)
+            (xy -0.625 0.85)
+            (xy -0.625 -0.55)
+          ) (width 0.01) (fill yes))
+      ))
   )
   (footprint "Capacitor_SMD:C_0805_2012Metric_Pad1.18x1.45mm_HandSolder" (layer "F.Cu")
@@
       (net 5 "Net-(D1-Pad2)") (pinfunction "A") (pintype "passive"))
     (model "${KICAD6_3DMODEL_DIR}/LED_SMD.3dshapes/LED_0805_2012Metric.wrl"
+      (offset (xyz 0 0 0))
+      (scale (xyz 1 1 1))
+      (rotate (xyz 0 0 0))
+    )
+  )
+  (footprint "Connector_Coaxial:U.FL_Molex_MCRF_73412-0110_Vertical" (layer "F.Cu")
+    (at 180.34 105.41)
+    (descr "Molex Microcoaxial RF Connectors (MCRF), mates Hirose U.FL, (http://www.molex.com/pdm_docs/sd/734120110_sd.pdf)")
+    (tags "mcrf hirose ufl u.fl microcoaxial")
+    (property "Sheetfile" "ESP32-aqs.kicad_sch")
+    (property "Sheetname" "")
+    (attr smd)
+    (fp_text reference "J3" (at 0 3.5) (layer "F.SilkS")
+      (effects (font (size 1 1) (thickness 0.15)))
+    )
+    (fp_text value "ufl connector" (at 0 -3.302) (layer "F.Fab")
+      (effects (font (size 1 1) (thickness 0.15)))
+    )
+    (fp_text user "${REFERENCE}" (at 0 3.5) (layer "F.Fab")
+      (effects (font (size 1 1) (thickness 0.15)))
+    )
+    (fp_line (start 1.5 1.5) (end 0.7 1.5) (layer "F.SilkS") (width 0.12))
+    (fp_line (start 1.5 1.3) (end 1.5 1.5) (layer "F.SilkS") (width 0.12))
+    (fp_line (start -1.3 1.5) (end -1.5 1.3) (layer "F.SilkS") (width 0.12))
+    (fp_line (start -1.5 -1.5) (end -0.7 -1.5) (layer "F.SilkS") (width 0.12))
+    (fp_line (start 0.7 -1.5) (end 1.5 -1.5) (layer "F.SilkS") (width 0.12))
+    (fp_line (start -0.7 1.5) (end -0.7 2) (layer "F.SilkS") (width 0.12))
+    (fp_line (start 1.5 -1.5) (end 1.5 -1.3) (layer "F.SilkS") (width 0.12))
+    (fp_line (start 0.7 1.5) (end 0.7 2) (layer "F.SilkS") (width 0.12))
+    (fp_line (start -0.7 1.5) (end -1.3 1.5) (layer "F.SilkS") (width 0.12))
+    (fp_line (start -1.5 -1.3) (end -1.5 -1.5) (layer "F.SilkS") (width 0.12))
+    (fp_line (start 2.5 -2.5) (end -2.5 -2.5) (layer "F.CrtYd") (width 0.05))
+    (fp_line (start -2.5 -2.5) (end -2.5 2.5) (layer "F.CrtYd") (width 0.05))
+    (fp_line (start 2.5 2.5) (end 2.5 -2.5) (layer "F.CrtYd") (width 0.05))
+    (fp_line (start -2.5 2.5) (end 2.5 2.5) (layer "F.CrtYd") (width 0.05))
+    (fp_line (start -1.3 -1.3) (end 1.3 -1.3) (layer "F.Fab") (width 0.1))
+    (fp_line (start -0.3 1.3) (end 0 1) (layer "F.Fab") (width 0.1))
+    (fp_line (start -1.3 1) (end -1 1.3) (layer "F.Fab") (width 0.1))
+    (fp_line (start 0 1) (end 0.3 1.3) (layer "F.Fab") (width 0.1))
+    (fp_line (start -1 1.3) (end 1.3 1.3) (layer "F.Fab") (width 0.1))
+    (fp_line (start 1.3 -1.3) (end 1.3 1.3) (layer "F.Fab") (width 0.1))
+    (fp_line (start -1.3 -1.3) (end -1.3 1) (layer "F.Fab") (width 0.1))
+    (fp_circle (center 0 0) (end 0 0.2) (layer "F.Fab") (width 0.1) (fill none))
+    (fp_circle (center 0 0) (end 0 0.125) (layer "F.Fab") (width 0.1) (fill none))
+    (fp_circle (center 0 0) (end 0.9 0) (layer "F.Fab") (width 0.1) (fill none))
+    (fp_circle (center 0 0) (end 0 0.05) (layer "F.Fab") (width 0.1) (fill none))
+    (pad "1" smd rect (at 0 1.5) (size 1 1) (layers "F.Cu" "F.Paste" "F.Mask")
+      (net 40 "Net-(J3-Pad1)") (pinfunction "In") (pintype "passive"))
+    (pad "2" smd rect (at 1.475 0) (size 1.05 2.2) (layers "F.Cu" "F.Paste" "F.Mask")
+      (net 2 "GND") (pinfunction "Ext") (pintype "passive"))
+    (pad "2" smd rect (at -1.475 0) (size 1.05 2.2) (layers "F.Cu" "F.Paste" "F.Mask")
+      (net 2 "GND") (pinfunction "Ext") (pintype "passive"))
+    (pad "2" smd rect (at 0 -1.5) (size 1 1) (layers "F.Cu" "F.Paste" "F.Mask")
+      (net 2 "GND") (pinfunction "Ext") (pintype "passive"))
+    (model "${KICAD6_3DMODEL_DIR}/Connector_Coaxial.3dshapes/U.FL_Molex_MCRF_73412-0110_Vertical.wrl"
       (offset (xyz 0 0 0))
       (scale (xyz 1 1 1))
@@
       (net 2 "GND") (pinfunction "GND") (pintype "input"))
     (pad "9" smd rect (at -8 -6.08 180) (size 2.54 1.524) (layers "F.Cu" "F.Paste" "F.Mask")
-      (net 40 "unconnected-(U4-Pad9)") (pinfunction "RF") (pintype "input+no_connect"))
+      (net 40 "Net-(J3-Pad1)") (pinfunction "RF") (pintype "input"))
     (pad "10" smd rect (at -8 -4 180) (size 2.54 1.524) (layers "F.Cu" "F.Paste" "F.Mask")
       (net 2 "GND") (pinfunction "GND") (pintype "input"))

Commit message: PCB design update
Parts:
- moved C4 55.1 mm to (182.4, 101.6), turned to -90 degrees
- moved C3 52.6 mm to (179.1, 101.6), turned to -90 degrees
- moved J3 29.4 mm to (186.5, 76.7)
- moved J2 27.7 mm to (188.2, 101.6), turned to 90 degrees
- moved U3 11.3 mm to (175.5, 100.6)
- moved J1 6.18 mm to (170.4, 78.0)
- moved D1 5.01 mm to (143.9, 78.2)
- moved TP1 5.01 mm to (128.3, 80.5)
- moved C2 5.01 mm to (134.3, 74.4)
- moved U1 5.01 mm to (136.4, 80.8)
- moved R1 4.21 mm to (143.8, 81.0)
- moved C1 3.08 mm to (134.2, 86.9)
- moved C9 3.05 mm to (206.8, 90.4)
- moved C8 2.18 mm to (203.5, 90.4)
- moved C6 1.59 mm to (138.9, 87.4)
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Routing:
- net GND: track 10.6 -> 92.6 mm, vias 0 -> 7
- net VIN: track 8.92 -> 79.8 mm, vias 0 -> 1
- net SCL: track 18.2 -> 46.8 mm, vias 0 -> 2
- net Net-(J3-Pad1): track 0.00 -> 23.9 mm
- net +3V3: track 112.4 -> 132.2 mm, vias 0 -> 7
- net SDA: track 22.0 -> 39.1 mm, vias 0 -> 2
- net TX: track 0.00 -> 16.8 mm
- net RX: track 0.00 -> 14.4 mm
- net RST: track 47.5 -> 53.0 mm
- net Net-(D1-Pad2): track 4.84 -> 2.86 mm
- net MOSI: track 19.6 -> 20.1 mm
- added copper zone on B.Cu, net GND
Other:
- board outline added: 107.6 x 52.7 mm

Commit message: PCB design
Parts:
- added H1: MountingHole, MountingHole:MountingHole_2.2mm_M2_ISO7380_Pad, F.Cu at (222.0, 61.2)
- added H2: MountingHole, MountingHole:MountingHole_2.2mm_M2_ISO7380_Pad, F.Cu at (222.0, 113.0)
- added H3: MountingHole, MountingHole:MountingHole_2.2mm_M2_ISO7380_Pad, F.Cu at (115.3, 113.0)
- added H4: MountingHole, MountingHole:MountingHole_2.2mm_M2_ISO7380_Pad, F.Cu at (115.6, 61.2)
- added SW1: RESET, Button_Switch_THT:SW_PUSH_6mm_H7.3mm, F.Cu at (137.7, 94.4)
- added SW2: BOOT, Button_Switch_THT:SW_PUSH_6mm_H7.3mm, F.Cu at (169.0, 101.4)
- J1: footprint Connector_PinHeader_2.54mm:PinHeader_1x04_P2.54mm_Vertical -> Connector_PinHeader_2.54mm:PinHeader_1x06_P2.54mm_Vertical
- J2: value Conn SEN55 -> JST connector SEN55; footprint Connector_PinHeader_2.54mm:PinHeader_1x05_P2.54mm_Vertical -> ESP32-aqs:JST_BM06B-GHS-TBT_LF__SN__N_
- moved J3 23.0 mm to (208.3, 69.3)
- moved J1 18.9 mm to (187.5, 69.8)
- moved R1 18.6 mm to (125.5, 77.7)
- moved TP1 17.7 mm to (122.9, 63.6), turned to 0 degrees
- moved U1 16.4 mm to (122.7, 71.7), turned to -90 degrees
- moved D1 15.2 mm to (129.0, 75.2), turned to -90 degrees
- moved C2 7.12 mm to (129.0, 69.6), turned to -90 degrees
- moved C5 4.32 mm to (142.5, 92.7)
- moved C1 4.32 mm to (134.2, 82.5)
- moved C3 4.32 mm to (179.1, 97.3)
- moved C4 4.32 mm to (182.4, 97.3)
- moved C6 4.32 mm to (138.9, 83.0)
- moved C7 4.32 mm to (142.5, 83.0)
- moved C8 4.32 mm to (203.5, 86.1)
- moved C9 4.32 mm to (206.8, 86.1)
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Connections:
- J1 pad 1: VIN -> unconnected-(J1-Pad1)
- J1 pad 4: GND -> VIN
Routing:
- net VIN: track 79.8 -> 129.7 mm
- net GND: track 92.6 -> 125.3 mm, vias 7 -> 6
- net TX: track 16.8 -> 34.6 mm
- net +3V3: track 132.2 -> 149.5 mm
- net RX: track 14.4 -> 31.6 mm
- net BOOT: track 0.00 -> 14.9 mm, vias 0 -> 1
- net (no net): track 9.47 -> 0.00 mm
- net EN: track 20.4 -> 26.2 mm
- net SCL: track 46.8 -> 44.0 mm
- net Net-(J3-Pad1): track 23.9 -> 26.6 mm
- net RST: track 53.0 -> 50.6 mm
- net SDA: track 39.1 -> 37.9 mm
- net MOSI: track 20.1 -> 19.0 mm
Other:
- board size 107.6 x 52.7 mm -> 110.7 x 55.9 mm

Commit message: PCB Design update
Routing:
- net GND: track 125.3 -> 164.2 mm
- net unconnected-(J2-PadS1): track 0.00 -> 9.95 mm
- net +3V3: track 149.5 -> 152.4 mm
- net SDA: track 37.9 -> 39.1 mm

Commit message: PCB design
Parts:
- added C10: 1µF, Capacitor_SMD:C_0805_2012Metric_Pad1.18x1.45mm_HandSolder, F.Cu at (206.8, 86.1)
- added R2: 4k7, Resistor_SMD:R_0805_2012Metric_Pad1.20x1.40mm_HandSolder, F.Cu at (206.8, 80.8)
- C8: value 1µF -> 100nF
- C9: value 1nF -> 1µF
- moved C9 3.30 mm to (210.1, 86.1), turned to 90 degrees
Connections:
- C9 pad 1: +3V3 -> GND
- C9 pad 2: GND -> ANT
- U4 pad 9: Net-(J3-Pad1) -> ANT
Routing:
- net ANT: track 0.00 -> 23.3 mm
- net Net-(J3-Pad1): track 26.6 -> 17.7 mm
- net GND: track 164.2 -> 167.5 mm
- net +3V3: track 152.4 -> 149.1 mm

Commit message: PCB Design
Parts:
- U2: value ESP32-WROOM-32 -> ESP32-WROOM-32-N8
- U4: value SX1276S8S+T-X1 -> DL-RFM95-868M
- moved H2 11.8 mm to (210.8, 109.2)
- moved H1 11.2 mm to (210.8, 61.2)
- moved H3 5.57 mm to (119.4, 109.2)
- moved H4 3.81 mm to (119.4, 61.2)
Other:
- board size 110.7 x 55.9 mm -> 98 x 53.3 mm

Commit message: PCB design geupdate
Parts:
- removed H1, H3: MountingHole, MountingHole:MountingHole_2.2mm_M2_ISO7380_Pad
- removed J1: UART Connector, Connector_PinHeader_2.54mm:PinHeader_1x06_P2.54mm_Vertical
- added J4: UART Connector, TerminalBlock_Phoenix:TerminalBlock_Phoenix_MPT-0,5-6-2.54_1x06_P2.54mm_Horizontal, F.Cu at (183.4, 80.8)
- SW1: value RESET -> TC-1102-B-C-B; footprint Button_Switch_THT:SW_PUSH_6mm_H7.3mm -> Button_Switch_THT:SW_PUSH_6mm
- SW2: value BOOT -> TC-1102-B-C-B; footprint Button_Switch_THT:SW_PUSH_6mm_H7.3mm -> Button_Switch_THT:SW_PUSH_6mm
- U2: value ESP32-WROOM-32-N8 -> ESP32-WROOM-32
- U4: value DL-RFM95-868M -> SX1276S8S+T-X1
- moved C8 57.5 mm to (149.6, 106.4), turned to 0 degrees
- moved H2 37.3 mm to (173.7, 105.2)
- moved U4 37.2 mm to (156.6, 95.6), turned to 0 degrees
- moved J3 34.3 mm to (173.9, 68.6)
- moved C9 34.3 mm to (177.4, 75.5)
- moved R2 33.7 mm to (173.9, 73.4)
- moved C10 32.6 mm to (177.7, 71.4), turned to -90 degrees
- moved U1 28.0 mm to (141.7, 92.3)
- moved C3 20.5 mm to (172.7, 77.7), turned to 180 degrees
- moved C4 19.8 mm to (172.7, 80.0), turned to 180 degrees
- moved R1 19.7 mm to (144.0, 84.6), turned to -90 degrees
- moved TP1 19.7 mm to (140.5, 72.6)
- moved H4 18.1 mm to (135.9, 68.6)
- moved U3 16.8 mm to (177.2, 79.5), turned to 90 degrees
- moved SW2 15.8 mm to (172.8, 86.1)
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Routing:
- net GND: track 167.5 -> 223.0 mm, vias 6 -> 2
- net +3V3: track 149.1 -> 110.5 mm, vias 7 -> 5
- net VIN: track 129.7 -> 91.5 mm
- net SDA: track 39.1 -> 61.0 mm, vias 2 -> 0
- net SCL: track 44.0 -> 65.1 mm
- net RST: track 50.6 -> 33.6 mm, vias 0 -> 2
- net MOSI: track 19.0 -> 34.3 mm, vias 2 -> 0
- net EN: track 26.2 -> 41.3 mm, vias 0 -> 1
- net TX: track 34.6 -> 19.8 mm, vias 0 -> 1
- net ANT: track 23.3 -> 35.1 mm, vias 0 -> 2
- net Net-(J3-In): track 17.7 -> 6.16 mm
- net RX: track 31.6 -> 22.6 mm, vias 0 -> 1
- net MISO: track 21.4 -> 30.3 mm
- net SCK: track 20.3 -> 24.6 mm
- net Net-(D1-A): track 3.16 -> 5.28 mm
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Other:
- board size 98 x 53.3 mm -> 54.1 x 41.9 mm

Commit message: PCB v2
Parts:
- added C11: 0.1µF, Capacitor_SMD:C_0805_2012Metric_Pad1.18x1.45mm_HandSolder, F.Cu at (135.9, 69.2)
- added C12: 0.1µF, Capacitor_SMD:C_0805_2012Metric_Pad1.18x1.45mm_HandSolder, F.Cu at (133.1, 69.2)
- added C13: 10µF, Capacitor_SMD:C_0805_2012Metric_Pad1.18x1.45mm_HandSolder, F.Cu at (135.9, 73.7)
- added C14: 0.1µF, Capacitor_SMD:C_0805_2012Metric_Pad1.18x1.45mm_HandSolder, F.Cu at (133.1, 73.7)
- added D2: LED, LED_SMD:LED_0805_2012Metric_Pad1.15x1.40mm_HandSolder, F.Cu at (129.5, 97.8)
- added D3: LED, LED_SMD:LED_0805_2012Metric_Pad1.15x1.40mm_HandSolder, F.Cu at (132.1, 97.8)
- added D4: D_Schottky, ESP32-aqs:SOD-123FL, F.Cu at (130.8, 94.0)
- added IC1: CP2102N-A02-GQFN24, ESP32-aqs:QFN50P400X400X80-25N, F.Cu at (128.8, 75.3)
- added J1: USB4085-GF-A_REVA4, ESP32-aqs:GCT_USB4085-GF-A_REVA4, F.Cu at (129.4, 86.4)
- added R6: 20k, Resistor_SMD:R_0805_2012Metric_Pad1.20x1.40mm_HandSolder, F.Cu at (133.1, 78.2)
- added R7: 47k, Resistor_SMD:R_0805_2012Metric_Pad1.20x1.40mm_HandSolder, F.Cu at (135.9, 78.2)
- added R8: 1k, Resistor_SMD:R_0805_2012Metric_Pad1.20x1.40mm_HandSolder, F.Cu at (132.1, 102.2)
- added R9: 1k, Resistor_SMD:R_0805_2012Metric_Pad1.20x1.40mm_HandSolder, F.Cu at (129.5, 102.2)
- U3: footprint Library:SGP41 -> ESP32-aqs:XDCR_SGP41-D-R4
- moved H4 8.39 mm to (127.5, 68.6)
Routing:
- net VBUS: track 0.00 -> 55.2 mm
- net +3V3: track 110.5 -> 163.7 mm, vias 5 -> 8
- net RX: track 22.6 -> 74.9 mm, vias 1 -> 2
- net TX: track 19.8 -> 70.3 mm, vias 1 -> 2
- net GND: track 223.0 -> 254.5 mm, vias 2 -> 3
- net TXLED: track 0.00 -> 30.2 mm, vias 0 -> 2
- net RXLED: track 0.00 -> 29.4 mm, vias 0 -> 2
- net D+: track 0.00 -> 19.7 mm, vias 0 -> 1
- net D-: track 0.00 -> 16.8 mm, vias 0 -> 1
- net Net-(IC1-VBUS): track 0.00 -> 9.03 mm
- net VIN: track 91.5 -> 100.5 mm, vias 1 -> 2
- net Net-(D2-A): track 0.00 -> 6.02 mm
- net Net-(D3-A): track 0.00 -> 5.52 mm
Other:
- board size 54.1 x 41.9 mm -> 62.8 x 41.9 mm
