File: Kicad/ESP32-aqs/ESP32-aqs.kicad_pcb (KiCad board)
At the start: 2 copper layers, 62.8 x 41.9 mm, 41 parts, among them IC1 CP2102N-A02-GQFN24, J1 USB4085-GF-A_REVA4, J2 JST connector SEN55, J3 ufl connector, J4 UART Connector, SW1 TC-1102-B-C-B, SW2 TC-1102-B-C-B, U1 LD1117S33TR_SOT223, U2 ESP32-WROOM-32, U3 SGP41-D-R4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

Commit message: pcb
Parts:
- moved R1 1.05 mm to (143.0, 84.8)
Connections:
- U2 pad 11: unconnected-(U2-IO26-Pad11) -> Callback
- U4 pad 14: unconnected-(U4-DIO0-Pad14) -> Callback
Routing:
- net Callback: track 0.00 -> 26.9 mm
- net GND: track 254.2 -> 237.7 mm, vias 3 -> 4
- net Net-(D1-A): track 5.28 -> 4.09 mm
- net +3V3: track 163.7 -> 162.9 mm

Commit message: pcb
Parts:
- moved D4 2.43 mm to (133.2, 94.0)
Routing:
- net VIN: track 100.5 -> 99.7 mm
- net TX: track 70.3 -> 69.8 mm
Other:
- board size 62.8 x 41.9 mm -> 63 x 41.9 mm
- board text added: "GND"
- board text added: "RX"
- board text added: "TX"
- board text added: "Vin"
- board text added: "x"

Commit message: pcb update
Parts:
- removed H4: MountingHole, MountingHole:MountingHole_2.2mm_M2_ISO7380_Pad
- added H1: MountingHole_Pad, MountingHole:MountingHole_2.2mm_M2_ISO7380_Pad, F.Cu at (127.5, 68.6)
- added J6: test point / jst connector, TerminalBlock_Phoenix:TerminalBlock_Phoenix_MPT-0,5-5-2.54_1x05_P2.54mm_Horizontal, F.Cu at (183.4, 85.1)
- added Q1: IRLML0030, Package_TO_SOT_SMD:SOT-23, F.Cu at (172.7, 73.6)
- added Q2: PMN48XP, Package_SO:TSOP-6_1.65x3.05mm_P0.95mm, F.Cu at (176.7, 69.7)
- added R10: 100k, Resistor_SMD:R_0805_2012Metric_Pad1.20x1.40mm_HandSolder, F.Cu at (176.0, 73.6)
- added R11: 100k, Resistor_SMD:R_0805_2012Metric_Pad1.20x1.40mm_HandSolder, F.Cu at (178.1, 73.6)
- added R12: 1M, Resistor_SMD:R_0805_2012Metric_Pad1.20x1.40mm_HandSolder, F.Cu at (173.5, 69.6)
- H2: value MountingHole -> MountingHole_Pad
- moved J3 31.2 mm to (173.5, 99.8), turned to 180 degrees
- moved C10 23.7 mm to (175.9, 95.0), turned to 90 degrees
- moved R2 21.6 mm to (173.6, 95.0), turned to -90 degrees
- moved C9 20.5 mm to (171.3, 95.0)
- moved J4 12.7 mm to (183.4, 68.1), turned to -90 degrees
- moved D4 8.42 mm to (135.9, 86.0), turned to -90 degrees
- moved C8 6.97 mm to (145.8, 100.6), turned to -90 degrees
- moved C4 5.15 mm to (177.8, 79.9), turned to -90 degrees
- moved U3 4.50 mm to (172.8, 79.9)
- moved J2 4.29 mm to (182.3, 102.4), turned to 0 degrees
- moved SW1 4.20 mm to (143.2, 103.6), turned to 180 degrees
- moved SW2 4.14 mm to (172.0, 90.2), turned to 90 degrees
- moved C3 3.59 mm to (175.6, 79.9), turned to -90 degrees
- moved D3 1.49 mm to (131.3, 99.1), turned to -90 degrees
- moved R8 1.40 mm to (131.3, 103.4)
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Connections:
- H2 pad 1: (no net) -> GND
- J4 pad 1: unconnected-(J4-Pin_1-Pad1) -> BAT
- U2 pad 10: unconnected-(U2-IO25-Pad10) -> VBAT
- U2 pad 12: unconnected-(U2-IO27-Pad12) -> READ_BAT
Routing:
- net VBAT: track 0.00 -> 32.6 mm, vias 0 -> 2
- net GND: track 237.7 -> 205.1 mm
- net READ_BAT: track 0.00 -> 27.5 mm, vias 0 -> 2
- net BAT: track 0.00 -> 25.1 mm
- net SDA: track 61.0 -> 42.1 mm
- net RX: track 75.1 -> 56.3 mm
- net VIN: track 99.7 -> 82.0 mm, vias 2 -> 1
- net TX: track 69.8 -> 57.5 mm
- net +3V3: track 162.9 -> 153.9 mm, vias 8 -> 5
- net ANT: track 35.1 -> 27.3 mm
- net Net-(Q2-D-Pad1): track 0.00 -> 7.62 mm
- net Net-(Q1-D): track 0.00 -> 7.30 mm
- net RXLED: track 29.4 -> 24.6 mm
- net SCL: track 65.1 -> 60.3 mm, vias 2 -> 1
- net VBUS: track 54.8 -> 50.6 mm
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Other:
- board size 63 x 41.9 mm -> 63.2 x 41.7 mm

Commit message: Add files via upload
Parts:
- removed R3: 10k, Resistor_SMD:R_0805_2012Metric_Pad1.20x1.40mm_HandSolder
- added C15: 0.1µF, Capacitor_SMD:C_0805_2012Metric_Pad1.18x1.45mm_HandSolder, F.Cu at (127.5, 98.5)
- added Q3: SS8050-G, ESP32-aqs:TRANS_SS8050-G, F.Cu at (132.0, 103.5)
- added Q4: SS8050-G, ESP32-aqs:TRANS_SS8050-G, F.Cu at (132.0, 99.7)
- added R13: 10k, Resistor_SMD:R_0805_2012Metric_Pad1.20x1.40mm_HandSolder, F.Cu at (127.5, 101.5)
- added R14: 10k, Resistor_SMD:R_0805_2012Metric_Pad1.20x1.40mm_HandSolder, F.Cu at (127.5, 104.5)
- C5: value 1µF -> 0.1µF
- R1: value 1kΩ -> 1k
- moved J4 12.8 mm to (183.4, 80.8), turned to 90 degrees
- moved J6 10.4 mm to (183.4, 95.5), turned to 90 degrees
- moved R8 9.34 mm to (129.5, 94.2)
- moved R9 9.34 mm to (127.2, 94.3)
- moved D2 5.64 mm to (132.0, 94.2)
- moved D3 5.64 mm to (134.2, 94.2)
- moved R1 0.32 mm to (143.0, 84.5)
Connections:
- IC1 pad 19: unconnected-(IC1-RTS-Pad19) -> RST
- IC1 pad 23: unconnected-(IC1-DTR-Pad23) -> DTR
Routing:
- net RST: track 33.6 -> 154.9 mm, vias 2 -> 3
- net BOOT: track 13.6 -> 60.8 mm, vias 1 -> 2
- net DTR: track 0.00 -> 42.5 mm, vias 0 -> 2
- net GND: track 205.1 -> 226.7 mm, vias 4 -> 5
- net Net-(D2-A): track 2.33 -> 15.6 mm
- net TX: track 57.5 -> 65.7 mm, vias 2 -> 3
- net SCL: track 60.3 -> 66.9 mm, vias 1 -> 2
- net EN: track 41.6 -> 47.0 mm
- net BAT: track 25.1 -> 21.1 mm
- net Net-(Q4-Pad1): track 0.00 -> 3.84 mm
- net VIN: track 82.0 -> 85.6 mm
- net Net-(Q3-Pad1): track 0.00 -> 3.31 mm
- net Net-(D3-A): track 2.32 -> 5.59 mm
- net RX: track 56.3 -> 59.5 mm
- net +3V3: track 153.9 -> 153.0 mm
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Other:
- board text added: "BAT"
- board text added: "SCL"
- board text added: "SDA"
- board text added: "VIN"
- board text removed: "Vin"
- board text removed: "x"

Commit message: PCB + BoM
Routing:
- net GND: track 226.7 -> 219.5 mm
- net VIN: track 85.6 -> 88.3 mm
- net RST: track 154.9 -> 153.8 mm
Other:
- board size 63.2 x 41.7 mm -> 63.9 x 41.7 mm
