File: Kicad/ESP32-aqs/ESP32-aqs.kicad_sch (KiCad schematic)
At the start: 28 parts, among them J2 JST connector SEN55, J3 ufl connector, J4 UART Connector, SW1 TC-1102-B-C-B, SW2 TC-1102-B-C-B, U1 LD1117S33TR_SOT223, U2 ESP32-WROOM-32, U3 SGP41-D-R4, U4 SX1276S8S+T-X1

Commit message: schematic v2
Parts:
- removed R1: 1kΩ, Resistor_SMD:R_0805_2012Metric_Pad1.20x1.40mm_HandSolder, symbol Device:R
- added C11, C12, C14: 0.1µF, Capacitor_SMD:C_0805_2012Metric_Pad1.18x1.45mm_HandSolder, symbol Device:C_Small
- added C13: 10µF, Capacitor_SMD:C_0805_2012Metric_Pad1.18x1.45mm_HandSolder, symbol Device:C_Small
- added D2, D3: LED, LED_SMD:LED_0805_2012Metric_Pad1.15x1.40mm_HandSolder, symbol Device:LED
- added D4: D_Schottky, ESP32-aqs:SOD-123FL, symbol Device:D_Schottky
- added IC1: CP2102N-A02-GQFN24, ESP32-aqs:QFN50P400X400X80-25N, symbol ESP32-aqs:CP2102N-A02-GQFN24
- added J1: USB4085-GF-A_REVA4, ESP32-aqs:GCT_USB4085-GF-A_REVA4, symbol ESP32-aqs:USB-C_Connector
- added R1, R8, R9: 1k, Resistor_SMD:R_0805_2012Metric_Pad1.20x1.40mm_HandSolder, symbol Device:R_Small
- added R6: 20k, Resistor_SMD:R_0805_2012Metric_Pad1.20x1.40mm_HandSolder, symbol Device:R_Small
- added R7: 47k, Resistor_SMD:R_0805_2012Metric_Pad1.20x1.40mm_HandSolder, symbol Device:R_Small
- U3: footprint Library:SGP41 -> ESP32-aqs:XDCR_SGP41-D-R4
Connections:
- net +3V3: now also C12.1, C14.1, IC1.5 (VIO), IC1.6 (VDD), R1.2, R8.1, R9.1
- net +5V: now also D4.1 (K)
- net GND: now also C11.2, C12.2, C13.2, C14.2, IC1.2 (GND_1), IC1.25 (GND_2), J1.A1 (GND), J1.A12 (GND), J1.B1 (GND), J1.B12 (GND), J1.P1 (SHELL), J1.P2 (SHELL), J1.P3 (SHELL), J1.P4 (SHELL), R7.2
- net RX: now also IC1.20 (RXD)
- net TX: now also IC1.21 (TXD)
- net at D1.2 (A): now also R1.1
- new net: IC1.8 (VBUS), R6.2, R7.1
- new net: D2.2 (A), R9.2
- new net: D3.2 (A), R8.2
- new net D+: IC1.3 (D+), J1.A6 (DP1), J1.B6 (DP2)
- new net D-: IC1.4 (D-), J1.A7 (DN1), J1.B7 (DN2)
- new net RXLED: D3.1 (K), IC1.13 (GPIO.1_/_RXT)
- new net TXLED: D2.1 (K), IC1.14 (GPIO.0_/_TXT)
- new net VBUS: C11.1, C13.1, D4.2 (A), IC1.7 (VREGIN), J1.A4 (VBUS), J1.A9 (VBUS), J1.B4 (VBUS), J1.B9 (VBUS), R6.1
- no-connect marks 32 -> 36
Other:
- moved on the sheet: C1, C10, C2, C3, C4, C5, C6, C7, C8, C9, D1, H2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

Commit message: pcb
Connections:
- net Callback: now reaches U4.14 (DIO0)
- net Callback: now also U2.11 (IO26)
- no-connect marks 36 -> 34
Changed lines of the file:
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@@
   (no_connect (at 187.96 68.58))
   (no_connect (at 187.96 73.66))
-  (no_connect (at 187.96 91.44))
   (no_connect (at 120.65 177.8))
   (no_connect (at 147.32 68.58))
@@
   (no_connect (at 187.96 96.52))
   (no_connect (at 254 104.14))
-  (no_connect (at 254 109.22))
   (no_connect (at 147.32 81.28))
   (no_connect (at 187.96 55.88))
@@
     (stroke (width 0) (type default))
   )
+  (wire (pts (xy 256.54 100.33) (xy 256.54 109.22))
+    (stroke (width 0) (type default))
+  )
   (wire (pts (xy 100.33 110.49) (xy 97.79 110.49))
     (stroke (width 0) (type default))
@@
   )
   (wire (pts (xy 100.33 128.27) (xy 97.79 128.27))
+    (stroke (width 0) (type default))
+  )
+  (wire (pts (xy 256.54 109.22) (xy 254 109.22))
     (stroke (width 0) (type default))
   )
@@
     )
   )
+  (global_label "Callback" (shape input) (at 187.96 91.44 0) (fields_autoplaced)
+    (effects (font (size 1.27 1.27)) (justify left))
+    (property "Intersheetrefs" "${INTERSHEET_REFS}" (at 199.1093 91.44 0)
+      (effects (font (size 1.27 1.27)) (justify left) hide)
+    )
+  )
   (global_label "TX" (shape input) (at 147.32 76.2 180) (fields_autoplaced)
     (effects (font (size 1.27 1.27)) (justify right))
@@
     )
   )
+  (global_label "Callback" (shape input) (at 256.54 100.33 0) (fields_autoplaced)
+    (effects (font (size 1.27 1.27)) (justify left))
+    (property "Intersheetrefs" "${INTERSHEET_REFS}" (at 267.6893 100.33 0)
+      (effects (font (size 1.27 1.27)) (justify left) hide)
+    )
+  )

Commit message: updated schematic
Parts:
- added Q1: IRLML0030, Package_TO_SOT_SMD:SOT-23, symbol Transistor_FET:IRLML0030
- added Q2: PMN48XP, Package_SO:TSOP-6_1.65x3.05mm_P0.95mm, symbol Transistor_FET:PMN48XP
- added R10, R11: 100k, Resistor_SMD:R_0805_2012Metric_Pad1.20x1.40mm_HandSolder, symbol Device:R_Small
- added R12: 1M, Resistor_SMD:R_0805_2012Metric_Pad1.20x1.40mm_HandSolder, symbol Device:R_Small
Connections:
- net GND: now also Q1.2 (S), R11.2
- net VBAT: now reaches U2.10 (IO25)
- net VBAT: now also R10.2, R11.1
- net BAT: now reaches J4.1 (Pin_1)
- net BAT: now also Q2.4 (S), R12.1
- new net: Q1.3 (D), Q2.3 (G), R12.2
- new net: Q2.1 (D), Q2.2 (D), Q2.5 (D), Q2.6 (D), R10.1
- no-connect marks 34 -> 32
Other:
- moved on the sheet: C1, C10, C11, C12, C13, C14, C2, C3, C4, C5, C6, C7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

Commit message: pcb update
Parts:
- removed H2, H4: MountingHole, MountingHole:MountingHole_2.2mm_M2_ISO7380_Pad, symbol Mechanical:MountingHole
- added H1, H2: MountingHole_Pad, MountingHole:MountingHole_2.2mm_M2_ISO7380_Pad, symbol Mechanical:MountingHole_Pad
- added J6: test point / jst connector, TerminalBlock_Phoenix:TerminalBlock_Phoenix_MPT-0,5-5-2.54_1x05_P2.54mm_Horizontal, symbol Connector:Screw_Terminal_01x05
Connections:
- net +5V: now also J6.1 (Pin_1)
- net GND: now also H1.1, H2.1, J6.2 (Pin_2), J6.5 (Pin_5)
- net SCL: now also J6.4 (Pin_4)
- net SDA: now also J6.3 (Pin_3)
- net READ_BAT: now reaches Q1.1 (G)
- net READ_BAT: now also U2.12 (IO27)
- no-connect marks 32 -> 31
Other:
- moved on the sheet: J2, R10, R11

Commit message: Add files via upload
Parts:
- removed R3: 10k, Resistor_SMD:R_0805_2012Metric_Pad1.20x1.40mm_HandSolder, symbol Device:R_Small
- added C15: 0.1µF, Capacitor_SMD:C_0805_2012Metric_Pad1.18x1.45mm_HandSolder, symbol Device:C_Small
- added Q3, Q4: SS8050-G, ESP32-aqs:TRANS_SS8050-G, symbol ESP32-aqs:SS8050-G
- added R13, R14: 10k, Resistor_SMD:R_0805_2012Metric_Pad1.20x1.40mm_HandSolder, symbol Device:R_Small
- C5: value 1µF -> 0.1µF
Connections:
- net BOOT: now also C15.1, Q4.3
- net EN: now also Q3.3
- net GND: now also C15.2
- net RST: now also IC1.19 (RTS), Q3.2, R13.1
- net DTR: now reaches IC1.23 (DTR)
- net DTR: now also Q4.2, R14.1
- new net: Q3.1, R14.2
- new net: Q4.1, R13.2
Other:
- moved on the sheet: C11, C12, C13, C14, IC1, R6, R7, SW2
