File: Kicad/ESP32-aqs.kicad_pcb (KiCad board)
At the start: 2 copper layers, 63.2 x 41.7 mm, 51 parts, among them IC1 CP2102N-A02-GQFN24, J1 USB4085-GF-A_REVA4, J2 JST connector SEN55, J3 ufl connector, J4 UART Connector, J6 test point / jst connector, Q1 IRLML0030, Q2 PMN48XP, Q3 SS8050-G, Q4 SS8050-G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

Commit message: PCB v3
Parts:
- removed J1: USB4085-GF-A_REVA4, ESP32-aqs:GCT_USB4085-GF-A_REVA4
- added J5: ~, ESP32-aqs:USB-TYPE-C-018, F.Cu at (131.0, 86.4)
- moved D4 0.61 mm to (136.5, 86.0)
Connections:
- U2 pad 11: Callback -> DIO1
- U2 pad 9: unconnected-(U2-IO33-Pad9) -> DIO0
- U4 pad 14: Callback -> DIO0
- U4 pad 15: unconnected-(U4-DIO1-Pad15) -> DIO1
Routing:
- net DIO0: track 0.00 -> 28.2 mm
- net Callback: track 26.9 -> 0.00 mm
- net DIO1: track 0.00 -> 24.0 mm, vias 0 -> 2
- net VBUS: track 50.6 -> 47.6 mm
- net D-: track 16.8 -> 19.3 mm, vias 1 -> 0
- net VIN: track 85.6 -> 87.4 mm
- net GND: track 226.7 -> 228.4 mm
- net D+: track 19.7 -> 20.8 mm, vias 1 -> 0
