File: Kicad/ESP32-aqs.kicad_sch (KiCad schematic)
At the start: 51 parts, among them IC1 CP2102N-A02-GQFN24, J1 USB4085-GF-A_REVA4, J2 JST connector SEN55, J3 ufl connector, J4 UART Connector, J6 test point / jst connector, Q1 IRLML0030, Q2 PMN48XP, Q3 SS8050-G, Q4 SS8050-G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

Commit message: PCB v3
Parts:
- removed J1: USB4085-GF-A_REVA4, ESP32-aqs:GCT_USB4085-GF-A_REVA4, symbol ESP32-aqs:USB-C_Connector
- added J5: ~, ESP32-aqs:USB-TYPE-C-018, symbol ESP32-aqs:USB-TYPE-C-018
Connections:
- net D+: now also J5.A6 (DP1), J5.B6 (DP2)
- net D-: now also J5.A7 (DN1), J5.B7 (DN2)
- net GND: now also J5.0 (SH), J5.1 (SH), J5.2 (SH), J5.3 (SH), J5.A1 (GND), J5.A12 (GND), J5.B1 (GND), J5.B12 (GND)
- net VBUS: now also J5.A4 (VBUS), J5.A9 (VBUS), J5.B4 (VBUS), J5.B9 (VBUS)
- net DIO1: now reaches U4.15 (DIO1)
- net DIO1: now also U2.11 (IO26)
- net DIO0: now reaches U2.9 (IO33)
- net DIO0: now also U4.14 (DIO0)
- removed net Callback: U2.11 (IO26), U4.14 (DIO0)
- no-connect marks 31 -> 29
